File: schematic_gprs_old.brd (EAGLE design)
At the start: 64.9 x 62 mm, 46 parts, among them J1 Jumper Alimentaciones, Q1 MOSFET-NCHANNEL2N7000, Q2 MOSFET-NCHANNEL2N7000, T1 BC547, X1 LTI-SASF54GT

Commit message: Resultado Final
PCB  a espera de revisión por tutor el día 18/02/2015
Changed lines of the file:
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@@
 <setting verticaltext="up"/>
 </settings>
-<grid distance="0.05" unitdist="inch" unit="inch" style="lines" multiple="1" display="no" altdistance="0.01" altunitdist="inch" altunit="inch"/>
+<grid distance="0.05" unitdist="inch" unit="mm" style="lines" multiple="1" display="no" altdistance="0.01" altunitdist="inch" altunit="mm"/>
 <layers>
 <layer number="1" name="Top" color="4" fill="1" visible="yes" active="yes"/>
@@
 <wire x1="54.57" y1="53.992" x2="60.698" y2="53.992" width="1.27" layer="1"/>
 <wire x1="60.698" y1="53.992" x2="61.5" y2="53.19" width="1.27" layer="1"/>
-<wire x1="52.79" y1="49.16" x2="52.79" y2="52.212" width="1.016" layer="1"/>
+<wire x1="52.79" y1="49.16" x2="52.79" y2="52.212" width="1.27" layer="1"/>
 <wire x1="52.79" y1="52.212" x2="54.57" y2="53.992" width="1.27" layer="1"/>
 <wire x1="51.29" y1="49.16" x2="51.29" y2="50.712" width="1.27" layer="1"/>
